File: Hardware/2DBarcodeScanner.brd (EAGLE design)
At the start: 44.5 x 25.4 mm, 58 parts, among them Q1 600mA/40V, Q2 600mA/40V, U1 3.3V

Commit message: Update silkscreen
Parts:
- removed U$16: (no value), output:3#3V0
- removed U$7: (no value), output:#3#3V#0
- added U$8: (no value), output:PWR0
- added U$9: (no value), output:#LED#0
- U$6: device output:#STAT#0 -> output:#STAT_LED#0
Changed lines of the file:
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@@
 <?xml version="1.0" encoding="utf-8"?>
 <!DOCTYPE eagle SYSTEM "eagle.dtd">
-<eagle version="9.5.2">
+<eagle version="9.6.2">
 <drawing>
 <settings>
@@
 <element name="U$2" library="output" package="#STAT_#0" value="" x="19.05" y="7.112" smashed="yes" rot="R270"/>
 <element name="U$3" library="output" package="STAT0" value="" x="20.955" y="5.715" smashed="yes"/>
-<element name="U$16" library="output" package="3#3V0" value="" x="10.16" y="22.733" smashed="yes" rot="R270"/>
 <element name="U$17" library="output" package="2D_BARCODE0" value="" x="15.367" y="12.319" smashed="yes"/>
 <element name="U$18" library="output" package="2D_BARCODE0" value="" x="24.892" y="19.939" smashed="yes" rot="MR0"/>
@@
 <element name="U$4" library="output" package="#SCAN#0" value="" x="31.115" y="15.24" smashed="yes" rot="R270"/>
 <element name="U$5" library="output" package="#BUZZ#0" value="" x="25.4" y="12.573" smashed="yes" rot="MR0"/>
-<element name="U$6" library="output" package="#STAT#0" value="" x="25.4" y="9.779" smashed="yes" rot="MR0"/>
-<element name="U$7" library="output" package="#3#3V#0" value="" x="7.62" y="19.558" smashed="yes" rot="MR270"/>
 <element name="R1" library="SparkFun-Resistors" package="0603" value="1k" x="23.876" y="2.54" smashed="yes">
 <attribute name="NAME" x="23.876" y="3.302" size="0.6096" layer="25" font="vector" ratio="20" align="bottom-center"/>
@@
 <attribute name="REV" value="" x="1.27" y="-10.16" size="1.778" layer="27" font="vector" ratio="15" display="off"/>
 </element>
+<element name="U$8" library="output" package="PWR0" value="" x="10.287" y="22.733" smashed="yes" rot="R270"/>
+<element name="U$9" library="output" package="#LED#0" value="" x="7.62" y="19.431" smashed="yes" rot="MR270"/>
+<element name="U$6" library="output" package="#STAT_LED#0" value="" x="25.4" y="9.779" smashed="yes" rot="MR0"/>
 </elements>
 <signals>

Commit message: QC Double Check Changes
Parts:
- renumbered JP1 to PWR_LED, U$1 to U2
Routing:
- net GND: track 3.85 -> 5.80 mm
Changed lines of the file:
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@@
 <?xml version="1.0" encoding="utf-8"?>
 <!DOCTYPE eagle SYSTEM "eagle.dtd">
-<eagle version="9.6.2">
+<eagle version="9.5.2">
 <drawing>
 <settings>
-<setting alwaysvectorfont="yes"/>
+<setting alwaysvectorfont="no"/>
 <setting verticaltext="up"/>
 </settings>
@@
 <layer number="45" name="Holes" color="7" fill="1" visible="yes" active="yes"/>
 <layer number="46" name="Milling" color="3" fill="1" visible="no" active="yes"/>
-<layer number="47" name="Measures" color="7" fill="1" visible="yes" active="yes"/>
+<layer number="47" name="Measures" color="7" fill="1" visible="no" active="yes"/>
 <layer number="48" name="Document" color="7" fill="1" visible="no" active="yes"/>
 <layer number="49" name="Reference" color="7" fill="1" visible="no" active="yes"/>
@@
 <attribute name="VALUE" x="2.54" y="12.7" size="0.762" layer="27" rot="R270" align="center"/>
 </element>
-<element name="U$1" library="SparkFun-Hardware" package="BARCODE_SCANNER_MOUNT" value="BARCODE_SCANNER_MOUNT" x="35.814" y="12.319" smashed="yes" rot="MR180">
+<element name="U2" library="SparkFun-Hardware" package="BARCODE_SCANNER_MOUNT" value="BARCODE_SCANNER_MOUNT" x="35.814" y="12.319" smashed="yes" rot="MR180">
 <attribute name="PROD_ID" value="LPA-14926" x="35.814" y="12.319" size="1.778" layer="28" rot="MR180" display="off"/>
 </element>
@@
 <attribute name="VALUE" x="20.32" y="3.302" size="0.6096" layer="27" font="vector" ratio="20" rot="R180"/>
 </element>
-<element name="JP1" library="SparkFun-Jumpers" package="SMT-JUMPER_2_NC_TRACE_SILK" package3d_urn="urn:adsk.eagle:package:39281/1" value="JUMPER-SMT_2_NC_TRACE_SILK" x="26.289" y="9.779" smashed="yes" rot="MR0">
+<element name="PWR_LED" library="SparkFun-Jumpers" package="SMT-JUMPER_2_NC_TRACE_SILK" package3d_urn="urn:adsk.eagle:package:39281/1" value="JUMPER-SMT_2_NC_TRACE_SILK" x="26.289" y="9.779" smashed="yes" rot="MR0">
 <attribute name="NAME" x="26.289" y="10.922" size="0.6096" layer="26" font="vector" ratio="20" rot="MR0" align="bottom-center"/>
 <attribute name="VALUE" x="26.289" y="8.636" size="0.6096" layer="28" font="vector" ratio="20" rot="MR0" align="top-center"/>
@@
 <via x="7.62" y="7.62" extent="1-16" drill="0.381"/>
 <contactref element="D2" pad="C"/>
-<wire x1="24.638" y1="16.637" x2="22.94" y2="16.03" width="0" layer="19" extent="1-1"/>
-<wire x1="29.718" y1="15.367" x2="24.638" y2="16.637" width="0" layer="19" extent="1-1"/>
+<wire x1="22.94" y1="16.03" x2="24.031" y2="16.03" width="0.2032" layer="1"/>
+<wire x1="24.031" y1="16.03" x2="24.638" y2="16.637" width="0.2032" layer="1"/>
 </signal>
 <signal name="3.3V" class="1">
@@
 <wire x1="31.58" y1="20.32" x2="31.58" y2="17.823" width="0.2032" layer="1"/>
 <wire x1="31.58" y1="17.823" x2="31.623" y2="17.78" width="0.2032" layer="1"/>
-<wire x1="33.782" y1="17.741" x2="33.821" y2="17.78" width="0.2032" layer="1"/>
 <wire x1="24.638" y1="15.494" x2="29.337" y2="15.494" width="0.2032" layer="16"/>
 <wire x1="29.337" y1="15.494" x2="31.623" y2="17.78" width="0.2032" layer="16"/>
@@
 </signal>
 <signal name="STATUS_OUT">
-<contactref element="JP1" pad="2"/>
+<contactref element="PWR_LED" pad="2"/>
 <contactref element="J4" pad="1"/>
 <wire x1="25.7683" y1="9.779" x2="23.622" y2="9.779" width="0.2032" layer="16"/>
@@
 </signal>
 <signal name="N$8">
-<contactref element="JP1" pad="1"/>
+<contactref element="PWR_LED" pad="1"/>
 <wire x1="26.8097" y1="9.779" x2="26.924" y2="9.6647" width="0.2032" layer="16"/>
 <wire x1="26.924" y1="9.6647" x2="26.924" y2="4.953" width="0.2032" layer="16"/>

Commit message: Update silkscreen
Parts:
- removed U$24, U$25: (no value), output:#TRIG_#0
- added U$1, U$7: (no value), output:##TRIG##0
Changed lines of the file:
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@@
 <?xml version="1.0" encoding="utf-8"?>
 <!DOCTYPE eagle SYSTEM "eagle.dtd">
-<eagle version="9.5.2">
+<eagle version="9.6.2">
 <drawing>
 <settings>
-<setting alwaysvectorfont="no"/>
+<setting alwaysvectorfont="yes"/>
 <setting verticaltext="up"/>
 </settings>
@@
 <element name="U$19" library="output" package="SCANNER0" value="" x="16.51" y="10.922" smashed="yes"/>
 <element name="U$21" library="output" package="#STAT_#0" value="" x="19.05" y="7.112" smashed="yes" rot="MR270"/>
-<element name="U$24" library="output" package="#TRIG_#0" value="" x="16.51" y="6.477" smashed="yes" rot="R270"/>
-<element name="U$25" library="output" package="#TRIG_#0" value="" x="16.51" y="6.477" smashed="yes" rot="MR270"/>
 <element name="U$28" library="output" package="#3#3V_#0" value="" x="13.97" y="6.35" smashed="yes" rot="R270"/>
 <element name="U$29" library="output" package="#3#3V_#0" value="" x="13.97" y="6.35" smashed="yes" rot="MR270"/>
@@
 <element name="U$9" library="output" package="#LED#0" value="" x="7.62" y="19.431" smashed="yes" rot="MR270"/>
 <element name="U$6" library="output" package="#STAT_LED#0" value="" x="25.4" y="9.779" smashed="yes" rot="MR0"/>
+<element name="U$1" library="output" package="##TRIG##0" value="" x="16.51" y="6.477" smashed="yes" rot="R270"/>
+<element name="U$7" library="output" package="##TRIG##0" value="" x="16.51" y="6.477" smashed="yes" rot="MR270"/>
 </elements>
 <signals>
