File: Hardware/2DBarcodeScanner.sch (EAGLE design)
At the start: 36 parts, among them Q1 600mA/40V, Q2 600mA/40V, U1 3.3V, U2 BARCODE_SCANNER_MOUNT

Commit message: Update version number and re-panelize v11
Other:
- note added: "v11"
- note removed: "v10"
Changed lines of the file:
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@@
 <?xml version="1.0" encoding="utf-8"?>
 <!DOCTYPE eagle SYSTEM "eagle.dtd">
-<eagle version="9.5.2">
+<eagle version="9.6.2">
 <drawing>
 <settings>
@@
 <text x="167.64" y="7.62" size="2.54" layer="94" font="vector">Nick Poole
 Revised By: Priyanka Makin</text>
-<text x="238.76" y="7.62" size="2.54" layer="94" font="vector">v10</text>
+<text x="238.76" y="7.62" size="2.54" layer="94" font="vector">v11</text>
 <text x="27.94" y="129.54" size="1.778" layer="94" font="vector">Vin Range: 2.5 - 6.0 V</text>
 </plain>

Commit message: Switch status LED from blue to green and change pull-up to 100 ohms
Parts:
- D2: value BLUE -> GREEN; device SparkFun-LED:LED-BLUE0603 -> SparkFun-LED:LED-GREEN0603
- R1: value 1k -> 100; device SparkFun-Resistors:1KOHM-0603-1/10W-1% -> SparkFun-Resistors:100OHM-0603-1/10W-1%
Changed lines of the file:
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@@
 <?xml version="1.0" encoding="utf-8"?>
 <!DOCTYPE eagle SYSTEM "eagle.dtd">
-<eagle version="9.6.2">
+<eagle version="9.5.2">
 <drawing>
 <settings>
@@
 <part name="GND12" library="SparkFun-PowerSymbols" deviceset="GND" device=""/>
 <part name="SUPPLY2" library="SparkFun-PowerSymbols" deviceset="3.3V" device=""/>
-<part name="R1" library="SparkFun-Resistors" deviceset="1KOHM" device="-0603-1/10W-1%" value="1k"/>
-<part name="D2" library="SparkFun-LED" deviceset="LED-BLUE" device="0603" value="BLUE"/>
+<part name="R1" library="SparkFun-Resistors" deviceset="100OHM" device="-0603-1/10W-1%" value="100"/>
+<part name="D2" library="SparkFun-LED" deviceset="LED-GREEN" device="0603" value="GREEN"/>
 <part name="FRAME1" library="SparkFun-Aesthetics" deviceset="FRAME-LETTER" device=""/>
 </parts>
