File: Hardware/Production/2DBarcodeScanner-Panel.brd (EAGLE design)
At the start: 154.4 x 117.3 mm, 690 parts, among them Q1 600mA/40V, Q10 600mA/40V, Q11 600mA/40V, Q12 600mA/40V, Q13 600mA/40V, Q14 600mA/40V, Q15 600mA/40V, Q16 600mA/40V, Q17 600mA/40V, Q18 600mA/40V, Q19 600mA/40V, Q2 600mA/40V, Q20 600mA/40V, Q21 600mA/40V, Q22 600mA/40V, Q23 600mA/40V, Q24 600mA/40V, Q3 600mA/40V, Q4 600mA/40V, Q5 600mA/40V, Q6 600mA/40V, Q7 600mA/40V, Q8 600mA/40V, Q9 600mA/40V, U1 3.3V, U10 3.3V, U11 BARCODE_SCANNER_MOUNT, U12 3.3V, U13 BARCODE_SCANNER_MOUNT, U14 3.3V, U15 BARCODE_SCANNER_MOUNT, U16 3.3V, U17 BARCODE_SCANNER_MOUNT, U18 3.3V, U19 BARCODE_SCANNER_MOUNT, U2 BARCODE_SCANNER_MOUNT, U20 3.3V, U21 BARCODE_SCANNER_MOUNT, U22 3.3V, U23 BARCODE_SCANNER_MOUNT, U24 3.3V, U3 BARCODE_SCANNER_MOUNT, U4 3.3V, U5 BARCODE_SCANNER_MOUNT, U6 3.3V, U7 BARCODE_SCANNER_MOUNT, U8 3.3V, U9 BARCODE_SCANNER_MOUNT

Commit message: Update version number and re-panelize v11
Parts:
- moved U$120 2.54 mm to (98.8, 31.0)
- moved U$121 2.54 mm to (98.8, 31.0)
- moved U$122 2.54 mm to (101.3, 31.0)
- moved U$123 2.54 mm to (101.3, 31.0)
- moved U$186 2.54 mm to (98.8, 56.9)
- moved U$187 2.54 mm to (98.8, 56.9)
- moved U$188 2.54 mm to (101.3, 56.9)
- moved U$189 2.54 mm to (101.3, 56.9)
- moved U$252 2.54 mm to (98.8, 82.8)
- moved U$253 2.54 mm to (98.8, 82.8)
- moved U$254 2.54 mm to (101.3, 82.8)
- moved U$255 2.54 mm to (101.3, 82.8)
- moved U$54 2.54 mm to (98.8, 5.08)
- moved U$55 2.54 mm to (98.8, 5.08)
- moved U$56 2.54 mm to (101.3, 5.08)
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Connections:
- net RXI: now also J3.9, J4.4; no longer J3.8, J4.5
- net RXI1: now also J5.4, J6.9; no longer J5.5, J6.8
- net RXI10: now also J32.4, J33.9; no longer J32.5, J33.8
- net RXI11: now also J35.4, J36.9; no longer J35.5, J36.8
- net RXI2: now also J8.4, J9.9; no longer J8.5, J9.8
- net RXI3: now also J11.4, J12.9; no longer J11.5, J12.8
- net RXI4: now also J14.4, J15.9; no longer J14.5, J15.8
- net RXI5: now also J17.4, J18.9; no longer J17.5, J18.8
- net RXI6: now also J20.4, J21.9; no longer J20.5, J21.8
- net RXI7: now also J23.4, J24.9; no longer J23.5, J24.8
- net RXI8: now also J26.4, J27.9; no longer J26.5, J27.8
- net RXI9: now also J29.4, J30.9; no longer J29.5, J30.8
- net TXO: now also J3.8, J4.5; no longer J3.9, J4.4
- net TXO1: now also J5.5, J6.8; no longer J5.4, J6.9
- net TXO10: now also J32.5, J33.8; no longer J32.4, J33.9
- net TXO11: now also J35.5, J36.8; no longer J35.4, J36.9
- net TXO2: now also J8.5, J9.8; no longer J8.4, J9.9
- net TXO3: now also J11.5, J12.8; no longer J11.4, J12.9
- net TXO4: now also J14.5, J15.8; no longer J14.4, J15.9
- net TXO5: now also J17.5, J18.8; no longer J17.4, J18.9
- net TXO6: now also J20.5, J21.8; no longer J20.4, J21.9
- net TXO7: now also J23.5, J24.8; no longer J23.4, J24.9
- net TXO8: now also J26.5, J27.8; no longer J26.4, J27.9
- net TXO9: now also J29.5, J30.8; no longer J29.4, J30.9
Routing:
- net RXI2: track 23.2 -> 21.6 mm
- net TXO5: track 21.6 -> 23.2 mm
- net RXI5: track 23.2 -> 21.6 mm
- net TXO8: track 21.6 -> 23.2 mm
- net TXO2: track 21.6 -> 23.2 mm
- net TXO11: track 21.6 -> 23.2 mm
- net TXO10: track 21.6 -> 23.2 mm
- net RXI8: track 23.2 -> 21.6 mm
- net RXI3: track 23.2 -> 21.6 mm
- net RXI11: track 23.2 -> 21.6 mm
- net TXO4: track 21.6 -> 23.2 mm
- net TXO3: track 21.6 -> 23.2 mm
- net RXI9: track 23.2 -> 21.6 mm
- net RXI6: track 23.2 -> 21.6 mm
- net RXI4: track 23.2 -> 21.6 mm
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Other:
- board text added: "v11"
- board text removed: "v10"

Commit message: Re-panelize for BOM change
Parts:
- D10, D12, D14, D16, D18, D2, D20, D22, D24, D4, D6, D8: value BLUE -> GREEN
- R1, R108, R18, R27, R36, R45, R54, R63, R72, R81, R90, R99: value 1k -> 100

Commit message: Add gerbers for new scanner
Parts:
- removed BUZZ10, BUZZ11, BUZZ8, BUZZ9, PWR10, PWR11, PWR8, PWR9, PWR_LED10, PWR_LED11, PWR_LED8, PWR_LED9: JUMPER-SMT_2_NC_TRACE_SILK, SparkFun-Jumpers:SMT-JUMPER_2_NC_TRACE_SILK
- removed C25, C26, C28, C29, C31, C32, C34, C35: 1.0uF, SparkFun-Capacitors:0603
- removed C27, C30, C33, C36: 0.1uF, SparkFun-Capacitors:0603
- removed D17, D19, D21, D23: RED, SparkFun-LED:LED-0603
- removed D18, D20, D22, D24: GREEN, SparkFun-LED:LED-0603
- removed FD33, FD34, FD35, FD36, FD37, FD38, FD39, FD40, FD41, FD42, FD43, FD44, FD45, FD46, FD47, FD48: FIDUCIALUFIDUCIAL, SparkFun-Aesthetics:FIDUCIAL-MICRO
- removed H17, H18, H19, H20, H21, H22, H23, H24: STAND-OFF, SparkFun-Hardware:STAND-OFF
- removed J25, J28, J31, J34: (no value), SparkFun-Connectors:USB-C-16P-2LAYER-PADS
- removed J26, J29, J32, J35: (no value), SparkFun-Connectors:1X06_NO_SILK
- removed J27, J30, J33, J36: (no value), SparkFun-Connectors:FPC_12_0.5MM
- removed LOGO25, LOGO28, LOGO31, LOGO34: OSHW-LOGOS, SparkFun-Aesthetics:OSHW-LOGO-S
- removed LOGO26, LOGO29, LOGO32, LOGO35: SFE_LOGO_FLAME.1_INCH, SparkFun-Aesthetics:SFE_LOGO_FLAME_.1
- removed LOGO27, LOGO30, LOGO33, LOGO36: SFE_LOGO_NAME.1_INCH, SparkFun-Aesthetics:SFE_LOGO_NAME_.1
- removed LS10, LS11, LS12, LS9: BUZZER-SMD, SparkFun-Electromechanical:BUZZER-CCV
- removed Q17, Q18, Q19, Q20, Q21, Q22, Q23, Q24: 600mA/40V, SparkFun-DiscreteSemi:SOT23-3
- removed R100, R101, R73, R74, R82, R83, R91, R92: 5.1k, SparkFun-Resistors:0603
- removed R102, R75, R84, R93: 10, SparkFun-Resistors:0603
- removed R103, R105, R76, R78, R85, R87, R94, R96: 10k, SparkFun-Resistors:0603
- removed R104, R106, R107, R77, R79, R80, R86, R88, R89, R95, R97, R98: 1k, SparkFun-Resistors:0603
- removed R108, R81, R90, R99: 100, SparkFun-Resistors:0603
- removed S10, S11, S12, S9: MOMENTARY-SWITCH-SPST-SMD-5.2MM-TALL, SparkFun-Switches:TACTILE_SWITCH_SMD_5.2MM
- removed U$177, U$183, U$199, U$205, U$221, U$227, U$243, U$249: (no value), output:#STAT_#0
- removed U$178, U$200, U$222, U$244: (no value), output:STAT0
- removed U$179, U$180, U$201, U$202, U$223, U$224, U$245, U$246: (no value), output:2D_BARCODE0
- removed U$181, U$203, U$225, U$247: (no value), output:SCANNER_BREAKOUT0
- removed U$182, U$204, U$226, U$248: (no value), output:SCANNER0
- removed U$184, U$185, U$206, U$207, U$228, U$229, U$250, U$251: (no value), output:#3#3V_#0
- removed U$186, U$187, U$208, U$209, U$230, U$231, U$252, U$253: (no value), output:#TX_#0
- removed U$188, U$189, U$210, U$211, U$232, U$233, U$254, U$255: (no value), output:#RX_#0
- removed U$190, U$191, U$212, U$213, U$234, U$235, U$256, U$257: (no value), output:#GND_#0
- removed U$192, U$214, U$236, U$258: (no value), output:#SCAN#0
- removed U$193, U$215, U$237, U$259: (no value), output:#BUZZ#0
- removed U$194, U$216, U$238, U$260: (no value), output:PWR0
- removed U$195, U$217, U$239, U$261: (no value), output:#LED#0
- removed U$196, U$218, U$240, U$262: (no value), output:#STAT_LED#0
- removed U$197, U$198, U$219, U$220, U$241, U$242, U$263, U$264: (no value), output:##TRIG##0
- removed U17, U19, U21, U23: BARCODE_SCANNER_MOUNT, SparkFun-Hardware:BARCODE_SCANNER_MOUNT
- removed U18, U20, U22, U24: 3.3V, SparkFun-IC-Power:SOT23-5
- U$10: device output:#STAT_#0 -> SCANNER_V2:SCANNER_V20
- U$100, U$122, U$144, U$166, U$34, U$56, U$78: device output:#RX_#0 -> output:#GND_#0
- U$101, U$123, U$145, U$167, U$35, U$57, U$79: device output:#RX_#0 -> output:#SCAN#0
- U$102, U$124, U$146, U$168, U$36, U$58, U$80: device output:#GND_#0 -> output:#BUZZ#0
- U$103, U$125, U$147, U$169, U$37, U$59, U$81: device output:#GND_#0 -> output:PWR0
- U$104, U$126, U$148, U$170, U$38, U$60, U$82: device output:#SCAN#0 -> output:#LED#0
- U$105, U$127, U$149, U$171, U$39, U$61, U$83: device output:#BUZZ#0 -> output:#STAT_LED#0
- U$106, U$128, U$150, U$172, U$40, U$62, U$84: device output:PWR0 -> output:##TRIG##0
- U$107, U$129, U$151, U$173, U$41, U$63, U$85: device output:#LED#0 -> output:##TRIG##0
- U$108, U$130, U$152, U$174, U$42, U$64, U$86: device output:#STAT_LED#0 -> SCANNER_V2:SCANNER_V20
- U$109, U$131, U$153, U$175, U$43, U$65, U$87: device output:##TRIG##0 -> BREAKOUT_V2:BREAKOUT_V20
- U$11: device output:STAT0 -> BREAKOUT_V2:BREAKOUT_V20
- U$110, U$132, U$154, U$176, U$44, U$66, U$88: device output:##TRIG##0 -> 2D_BARCODE_SCANNER:2D_BARCODE_SCANNER0
- U$114, U$13, U$136, U$158, U$48, U$70, U$92: device output:2D_BARCODE0 -> output:#STAT_#0
- U$115, U$137, U$159, U$49, U$71, U$93: device output:SCANNER_BREAKOUT0 -> output:#3#3V_#0
- U$116, U$138, U$160, U$19, U$50, U$72, U$94: device output:SCANNER0 -> output:#3#3V_#0
- U$117, U$139, U$161, U$51, U$73, U$95: device output:#STAT_#0 -> output:#TX_#0
- U$118, U$140, U$162, U$22, U$52, U$74, U$96: device output:#3#3V_#0 -> output:#TX_#0
- U$119, U$141, U$163, U$23, U$53, U$75, U$97: device output:#3#3V_#0 -> output:#RX_#0
- U$12: device output:2D_BARCODE0 -> 2D_BARCODE_SCANNER:2D_BARCODE_SCANNER0
- U$120, U$142, U$164, U$24, U$54, U$76, U$98: device output:#TX_#0 -> output:#RX_#0
- U$121, U$143, U$165, U$25, U$55, U$77, U$99: device output:#TX_#0 -> output:#GND_#0
- U$14: device output:SCANNER_BREAKOUT0 -> output:STAT0
- U$15: device output:SCANNER0 -> output:2D_BARCODE0
- U$18: device output:2D_BARCODE0 -> output:#3#3V_#0
- U$20: device output:SCANNER_BREAKOUT0 -> output:#TX_#0
- moved U$60 117.3 mm to (7.62, 45.3), flipped to the bottom
- moved U$49 104.3 mm to (14.0, 32.3), flipped to the top, turned to 270 degrees
- moved U$64 103.6 mm to (15.4, 37.0), flipped to the top
- moved U$51 102.9 mm to (8.89, 31.0), flipped to the top
- moved U$56 98.7 mm to (6.35, 32.0), flipped to the bottom
- moved U$52 98.1 mm to (8.89, 31.0), flipped to the bottom
- moved U$48 96.6 mm to (19.1, 33.0), turned to 270 degrees
- moved U$55 96.3 mm to (6.35, 32.0), flipped to the top
- moved U$59 95.9 mm to (10.3, 48.6), flipped to the top
- moved U$53 95.7 mm to (11.4, 31.0), flipped to the top
- moved U$50 94.9 mm to (14.0, 32.3), flipped to the bottom, turned to 270 degrees
- moved C7 93.6 mm to (15.2, 48.0)
- moved C8 93.6 mm to (15.2, 42.2)
- moved J7 93.6 mm to (6.35, 38.6)
- moved U6 93.6 mm to (15.2, 45.1)
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Connections:
- removed net !SCAN_TRIGGER!10: C33.1, J32.2, J33.1, S11.3
- removed net !SCAN_TRIGGER!11: C36.1, J35.2, J36.1, S12.3
- removed net !SCAN_TRIGGER!8: C27.1, J26.2, J27.1, S9.3
- removed net !SCAN_TRIGGER!9: C30.1, J29.2, J30.1, S10.3
- removed net 3.3V10: C32.1, J32.3, J33.11, PWR10.2, Q22.3, R93.2, U22.5
- removed net 3.3V11: C35.1, J35.3, J36.11, PWR11.2, Q24.3, R102.2, U24.5
- removed net 3.3V8: C26.1, J26.3, J27.11, PWR8.2, Q18.3, R75.2, U18.5
- removed net 3.3V9: C29.1, J29.3, J30.11, PWR9.2, Q20.3, R84.2, U20.5
- removed net 5V10: C31.1, J31.VBUS1, J31.VBUS2, U22.1, U22.3
- removed net 5V11: C34.1, J34.VBUS1, J34.VBUS2, U24.1, U24.3
- removed net 5V8: C25.1, J25.VBUS1, J25.VBUS2, U18.1, U18.3
- removed net 5V9: C28.1, J28.VBUS1, J28.VBUS2, U20.1, U20.3
- removed net BUZZER10: J33.4, R95.1
- removed net BUZZER11: J36.4, R104.1
- removed net BUZZER8: J27.4, R77.1
- removed net BUZZER9: J30.4, R86.1
- removed net CC17: J25.A5, R74.2
- removed net CC18: J25.B5, R73.2
- removed net CC19: J28.A5, R83.2
- removed net CC20: J28.B5, R82.2
- removed net CC21: J31.A5, R92.2
- removed net CC22: J31.B5, R91.2
- removed net CC23: J34.A5, R101.2
- removed net CC24: J34.B5, R100.2
- removed net GND10: C31.2, C32.2, C33.2, D21.C, D22.C, J31.GND, J31.GND2, J32.6, J33.10, Q21.2, R91.1, R92.1, R94.1, R96.1, S11.1, U22.2
- removed net GND11: C34.2, C35.2, C36.2, D23.C, D24.C, J34.GND, J34.GND2, J35.6, J36.10, Q23.2, R100.1, R101.1, R103.1, R105.1, S12.1, U24.2
- removed net GND8: C25.2, C26.2, C27.2, D17.C, D18.C, J25.GND, J25.GND2, J26.6, J27.10, Q17.2, R73.1, R74.1, R76.1, R78.1, S9.1, U18.2
- removed net GND9: C28.2, C29.2, C30.2, D19.C, D20.C, J28.GND, J28.GND2, J29.6, J30.10, Q19.2, R82.1, R83.1, R85.1, R87.1, S10.1, U20.2
- removed net N$100: LS12.-, Q23.3
- removed net N$101: Q23.1, R103.2, R104.2
- removed net N$102: Q24.2, R108.2
- removed net N$103: Q24.1, R105.2, R106.2
- removed net N$104: D24.A, PWR_LED11.1
- removed net N$105: BUZZ11.2, R102.1
- removed net N$106: BUZZ11.1, LS12.+
- removed net N$107: PWR11.1, R107.1
- removed net N$108: D23.A, R107.2
- removed net N$73: LS9.-, Q17.3
- removed net N$74: Q17.1, R76.2, R77.2
- removed net N$75: Q18.2, R81.2
- removed net N$76: Q18.1, R78.2, R79.2
- removed net N$77: D18.A, PWR_LED8.1
- removed net N$78: BUZZ8.2, R75.1
- removed net N$79: BUZZ8.1, LS9.+
- removed net N$80: PWR8.1, R80.1
- removed net N$81: D17.A, R80.2
- removed net N$82: LS10.-, Q19.3
- removed net N$83: Q19.1, R85.2, R86.2
- removed net N$84: Q20.2, R90.2
- removed net N$85: Q20.1, R87.2, R88.2
- removed net N$86: D20.A, PWR_LED9.1
- removed net N$87: BUZZ9.2, R84.1
- removed net N$88: BUZZ9.1, LS10.+
- removed net N$89: PWR9.1, R89.1
- removed net N$90: D19.A, R89.2
- removed net N$91: LS11.-, Q21.3
- removed net N$92: Q21.1, R94.2, R95.2
- removed net N$93: Q22.2, R99.2
- removed net N$94: Q22.1, R96.2, R97.2
- removed net N$95: D22.A, PWR_LED10.1
- removed net N$96: BUZZ10.2, R93.1
- removed net N$97: BUZZ10.1, LS11.+
- removed net N$98: PWR10.1, R98.1
- removed net N$99: D21.A, R98.2
- removed net RXI10: J32.4, J33.9
- removed net RXI11: J35.4, J36.9
- removed net RXI8: J26.4, J27.9
- removed net RXI9: J29.4, J30.9
- removed net STATUS_LED10: J33.3, R97.1
- removed net STATUS_LED11: J36.3, R106.1
- removed net STATUS_LED8: J27.3, R79.1
- removed net STATUS_LED9: J30.3, R88.1
- removed net STATUS_OUT10: J32.1, PWR_LED10.2, R99.1
- removed net STATUS_OUT11: J35.1, PWR_LED11.2, R108.1
- removed net STATUS_OUT8: J26.1, PWR_LED8.2, R81.1
- removed net STATUS_OUT9: J29.1, PWR_LED9.2, R90.1
- removed net TXO10: J32.5, J33.8
- removed net TXO11: J35.5, J36.8
- removed net TXO8: J26.5, J27.8
- removed net TXO9: J29.5, J30.8
- removed net USB_N10: J31.A7, J31.B7, J33.7
- removed net USB_N11: J34.A7, J34.B7, J36.7
- removed net USB_N8: J25.A7, J25.B7, J27.7
- removed net USB_N9: J28.A7, J28.B7, J30.7
- removed net USB_P10: J31.A6, J31.B6, J33.6
- removed net USB_P11: J34.A6, J34.B6, J36.6
- removed net USB_P8: J25.A6, J25.B6, J27.6
- removed net USB_P9: J28.A6, J28.B6, J30.6
Routing:
- net 3.3V9: track 79.0 -> 0.00 mm, vias 3 -> 0
- net 3.3V10: track 79.0 -> 0.00 mm, vias 3 -> 0
- net 3.3V8: track 79.0 -> 0.00 mm, vias 3 -> 0
- net 3.3V11: track 79.0 -> 0.00 mm, vias 3 -> 0
- net 5V8: track 34.5 -> 0.00 mm, vias 3 -> 0
- net 5V11: track 34.5 -> 0.00 mm, vias 3 -> 0
- net 5V10: track 34.5 -> 0.00 mm, vias 3 -> 0
- net 5V9: track 34.5 -> 0.00 mm, vias 3 -> 0
- net USB_P10: track 27.5 -> 0.00 mm, vias 2 -> 0
- net USB_P9: track 27.5 -> 0.00 mm, vias 2 -> 0
- net USB_P11: track 27.5 -> 0.00 mm, vias 2 -> 0
- net USB_P8: track 27.5 -> 0.00 mm, vias 2 -> 0
- net !SCAN_TRIGGER!9: track 27.5 -> 0.00 mm, vias 2 -> 0
- net !SCAN_TRIGGER!8: track 27.5 -> 0.00 mm, vias 2 -> 0
- net !SCAN_TRIGGER!11: track 27.5 -> 0.00 mm, vias 2 -> 0
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- removed copper zone on layer 1, net GND10
- removed copper zone on layer 16, net GND10
- removed copper zone on layer 1, net GND11
- removed copper zone on layer 16, net GND11
- removed copper zone on layer 1, net GND8
- removed copper zone on layer 16, net GND8
- removed copper zone on layer 1, net GND9
- removed copper zone on layer 16, net GND9
Other:
- board size 154.4 x 117.3 mm -> 117.1 x 116.8 mm
